Commit message: another wqy, memory allocation

File: jetsonNano/ros2_ws/src/controller/urdf/robomaster.urdf (robot description, URDF)
Before this commit: robot example_robot, 3 links, 2 joints
Joints:
- joint sensor_joint_back: child PING_sensor_back_link -> /KPING_sensor_back_link
- joint sensor_joint_front: child PING_sensor_front_link -> /PING_sensor_front_link
